File: PCB_Files/WS2812B_or_SK6812/WS2812B-HueStrip.brd (EAGLE design)
At the start: 58 x 36 mm, 19 parts

Commit message: fixed design
Parts:
- R1, R2, R3, R4, R5: device rcl:0204/7 -> diyHue:MULTI_RESISTOR
- U$1: device buck-converter:BUCK_CONVERTER_TE818 -> diyHue:BUCK_CONVERTER_TE818
Connections:
- net +3V3: now also R1.2@1, R1.2@2, R2.2@1, R2.2@2, R4.2@1, R4.2@2, R5.2@1, R5.2@2; no longer R1.2, R2.2, R4.2, R5.2
- net BTN1: now also R1.1@1, R1.1@2; no longer R1.1
- net BTN2: now also R2.1@1, R2.1@2; no longer R2.1
- net BTN3: now also R4.1@1, R4.1@2; no longer R4.1
- net BTN4: now also R5.1@1, R5.1@2; no longer R5.1
- net N$4: now also R3.2@1, R3.2@2; no longer R3.2
- net WS2812B-DATA: now also R3.1@1, R3.1@2; no longer R3.1
Routing:
- net +3V3: track 21.5 -> 39.3 mm
- net N$4: track 3.54 -> 6.08 mm
- net BTN4: track 13.0 -> 15.6 mm
- net BTN3: track 21.0 -> 23.6 mm
- net BTN2: track 15.4 -> 18.0 mm
- net BTN1: track 19.6 -> 22.1 mm
- net WS2812B-DATA: track 24.3 -> 26.8 mm
