File: PCB_Files/WS2812B_or_SK6812/WS2812B-HueStrip.brd (EAGLE design)
At the start: 58 x 36 mm, 19 parts

Commit message: Updated gerber Files to fix breaking bug
the original design had some errors that were only found after they were ordered. Those bugs hab been fixed.
Also there were new pictures exported of the design and schematic
Parts:
- added R6: 100R, diyHue:MULTI_RESISTOR
- moved R3 11.5 mm to (42.2, 14.2), turned to 90 degrees
Connections:
- removed net N$4: R3.2@1, R3.2@2, WEMOS1.RX
- new net N$2: R3.2@1, R3.2@2, WEMOS1.D5
- new net N$3: R6.2@1, R6.2@2, WEMOS1.RX
- net WS2812B-DATA: now also R6.1@1, R6.1@2
Routing:
- net N$3: track 0.00 -> 13.6 mm
- net N$2: track 0.00 -> 7.27 mm
- net N$4: track 6.08 -> 0.00 mm
- net WS2812B-DATA: track 26.8 -> 22.4 mm
Other:
- board text added: "D5"
- board text added: "RX"
- board text added: "Select RX or D5 as OUPUT"
